File: stm32 prototype.sch (KiCad schematic (older format))
At the start: 135 parts, among them J1 USB_B_Mini, J2 Conn_01x06, J3 Conn_01x02, J4 Conn_01x10, Q1 Q_NMOS_GSD, Q2 Q_NMOS_GSD, Q3 Q_NMOS_GSD, Q4 Q_NMOS_GSD, Q5 Q_NMOS_GSD, Q6 Q_NMOS_GSD, Q7 Q_NMOS_GSD, Q8 Q_NMOS_GSD, Q9 Q_NMOS_GSD, U1 FT232RL, U2 W25Q128JV-DTR, U3 STM32F407VGTx, U4 LD1117S33TR, U5 ESP32, U6 IS25LP016D-JNLE-TR, U7 TPS62203DBVR, Y1 Crystal_GND24, Y2 Crystal_GND24, Y3 Crystal_GND23

Commit message: began switching to esp32-wroom module
Parts:
- removed C19, C20, C21, C25, C26, C28, C29, C31, C33, C36, C37: 0.1uF, Capacitors_SMD:C_0603, symbol Device:C
- removed C22: 10uF, Capacitors_SMD:C_0603, symbol Device:C
- removed C23, C27: NC, Capacitors_SMD:C_0603, symbol Device:C
- removed C24: 1uF, Capacitors_SMD:C_0603, symbol Device:C
- removed C30: 10nF, Capacitors_SMD:C_0603, symbol Device:C
- removed C32: 3.3nF, Capacitors_SMD:C_0603, symbol Device:C
- removed C34, C35: C, Capacitors_SMD:C_0603, symbol Device:C
- removed J3: Conn_01x02, connectors_mdg:SMA_SMD_Jack_Straight, symbol Connector_Generic:Conn_01x02
- removed L1: 2.0nH, Inductors_SMD:L_0402, symbol Device:L
- removed L2: L, Inductors_SMD:L_0402, symbol Device:L
- removed Q9: Q_NMOS_GSD, TO_SOT_Packages_SMD:SOT-323_SC-70, symbol Device:Q_NMOS_GSD
- removed R29, R30, R31, R32, R33, R38, R39: 0R, Resistors_SMD:R_0603, symbol Device:R
- removed R37: 499R, Resistors_SMD:R_0603, symbol Device:R
- removed R53: 1MR, Resistors_SMD:R_0603, symbol Device:R
- removed U5: ESP32, ESP32-footprints-Lib:ESP32, symbol ESP32-footprints-Shem-Lib:ESP32
- removed U6: IS25LP016D-JNLE-TR, Housings_SOIC:SOIC-8_3.9x4.9mm_Pitch1.27mm, symbol flash_memory_mdg:IS25LP016D-JNLE-TR
- removed Y2: Crystal_GND24, Crystals:Crystal_SMD_SeikoEpson_TSX3225-4pin_3.2x2.5mm, symbol Device:Crystal_GND24
- removed Y3: Crystal_GND23, Crystals:Crystal_SMD_SeikoEpson_MC146-4pin_6.7x1.5mm, symbol Device:Crystal_GND23
- added J3: Conn_02x08_Top_Bottom, Pin_Headers:Pin_Header_Straight_2x08_Pitch2.54mm, symbol Connector_Generic:Conn_02x08_Top_Bottom
- added J5: Conn_02x04_Top_Bottom, Pin_Headers:Pin_Header_Straight_2x04_Pitch2.54mm, symbol Connector_Generic:Conn_02x04_Top_Bottom
- added Q10, Q9: 2N2219, TO_SOT_Packages_SMD:SOT-323_SC-70, symbol Transistor_BJT:2N2219
- added SW1: SW_Push, digikey-footprints:Switch_Tactile_SMD_B3U-1000P, symbol Switch:SW_Push
- added U5: ESP32-WROOM, ESP32-footprints-Lib:ESP32-WROOM, symbol ESP32-footprints-Shem-Lib:ESP32-WROOM
- R25: value 10K -> 12k
- R26: value 20k -> 12k
- R27: value 0R -> 12k
- R28: value 0R -> 470R
Connections:
- net labels added: ESP_EN, ESP_GPIO_0, FTDI_ES_DTR, FTDI_ES_RTS, FTDI_ES_RXD, FTDI_ES_TXD, FTDI_ST_DTR, FTDI_ST_RTS, FTDI_ST_RXD, FTDI_ST_TXD, ST_ESP_RXD, ST_ESP_TXD
- net labels removed: ESP32_CHIP_ENABLE, ESP32_POWER_ENABLE, ESP32_RXD, ESP32_TXD, ESP32_VOLTAGE_SENSE, FTDI_RTS, FTDI_RXD, FTDI_TXD, SD_CLK, SD_CMD, SD_DATA_0, SD_DATA_1, SD_DATA_2, SD_DATA_3
- wire segments 250 -> 203
Other:
- moved on the sheet: J4

Commit message: added push button to stm32, worked on some layout
Parts:
- removed SW1: SW_Push, digikey-footprints:Switch_Tactile_SMD_B3U-1000P, symbol Switch:SW_Push
- added D14: LED, LEDs:LED_1206, symbol Device:LED
- added Q11: Q_NMOS_GSD, TO_SOT_Packages_SMD:SOT-323_SC-70, symbol Device:Q_NMOS_GSD
- added R29: 330R, Resistors_SMD:R_0603, symbol Device:R
- added R30: 10K, Resistors_SMD:R_0603, symbol Device:R
- added R31: 12k, Resistors_SMD:R_0603, symbol Device:R
- added R32: 470R, Resistors_SMD:R_0603, symbol Device:R
- added SW1, SW2: SW_Push, switches_mdg:Switch_Tactile_6x6mm_Vertical_SMD_MJTP1230, symbol switches_mdg:SW_Push
Connections:
- net labels removed: FTDI_DTR
- wire segments 203 -> 210
- no-connect marks 0 -> 1
Other:
- moved on the sheet: J4
Changed lines of the file:
@@
 L Connector_Generic:Conn_01x10 J4
 U 1 1 5C3119D0
-P 7300 12550
-F 0 "J4" H 7380 12542 50  0000 L CNN
-F 1 "Conn_01x10" H 7380 12451 50  0000 L CNN
-F 2 "Pin_Headers:Pin_Header_Straight_1x10_Pitch2.54mm" H 7300 12550 50  0001 C CNN
-F 3 "~" H 7300 12550 50  0001 C CNN
-	1    7300 12550
+P 9600 11500
+F 0 "J4" H 9680 11492 50  0000 L CNN
+F 1 "Conn_01x10" H 9680 11401 50  0000 L CNN
+F 2 "Pin_Headers:Pin_Header_Straight_1x10_Pitch2.54mm" H 9600 11500 50  0001 C CNN
+F 3 "~" H 9600 11500 50  0001 C CNN
+	1    9600 11500
 	1    0    0    -1
 $EndComp
@@
 Text GLabel 6800 10750 2    50   Input ~ 0
 FTDI_CBUS4
-Text GLabel 7100 12150 0    50   Input ~ 0
-FTDI_DTR
-Text GLabel 7100 12250 0    50   Input ~ 0
+Text GLabel 9400 11200 0    50   Input ~ 0
 FTDI_RI
-Text GLabel 7100 12350 0    50   Input ~ 0
+Text GLabel 9400 11300 0    50   Input ~ 0
 FTDI_DCR
-Text GLabel 7100 12450 0    50   Input ~ 0
+Text GLabel 9400 11400 0    50   Input ~ 0
 FTDI_DCD
-Text GLabel 7100 12550 0    50   Input ~ 0
+Text GLabel 9400 11500 0    50   Input ~ 0
 FTDI_CBUS4
-Text GLabel 7100 12650 0    50   Input ~ 0
+Text GLabel 9400 11600 0    50   Input ~ 0
 FTDI_CBUS2
-Text GLabel 7100 12750 0    50   Input ~ 0
+Text GLabel 9400 11700 0    50   Input ~ 0
 FTDI_CBUS3
 $Comp
 L power:+5V #PWR0155
 U 1 1 5C3158AD
-P 7100 12850
-F 0 "#PWR0155" H 7100 12700 50  0001 C CNN
-F 1 "+5V" V 7115 12978 50  0000 L CNN
-F 2 "" H 7100 12850 50  0001 C CNN
-F 3 "" H 7100 12850 50  0001 C CNN
-	1    7100 12850
+P 9400 11800
+F 0 "#PWR0155" H 9400 11650 50  0001 C CNN
+F 1 "+5V" V 9415 11928 50  0000 L CNN
+F 2 "" H 9400 11800 50  0001 C CNN
+F 3 "" H 9400 11800 50  0001 C CNN
+	1    9400 11800
 	0    -1   -1   0
 $EndComp
@@
 L power:+3.3V #PWR0156
 U 1 1 5C315DEA
-P 7100 12950
-F 0 "#PWR0156" H 7100 12800 50  0001 C CNN
-F 1 "+3.3V" V 7115 13078 50  0000 L CNN
-F 2 "" H 7100 12950 50  0001 C CNN
-F 3 "" H 7100 12950 50  0001 C CNN
-	1    7100 12950
+P 9400 11900
+F 0 "#PWR0156" H 9400 11750 50  0001 C CNN
+F 1 "+3.3V" V 9415 12028 50  0000 L CNN
+F 2 "" H 9400 11900 50  0001 C CNN
+F 3 "" H 9400 11900 50  0001 C CNN
+	1    9400 11900
 	0    -1   -1   0
 $EndComp
@@
 L power:GND #PWR0157
 U 1 1 5C316BFC
-P 7100 13050
-F 0 "#PWR0157" H 7100 12800 50  0001 C CNN
-F 1 "GND" H 7105 12877 50  0000 C CNN
-F 2 "" H 7100 13050 50  0001 C CNN
-F 3 "" H 7100 13050 50  0001 C CNN
-	1    7100 13050
+P 9400 12000
+F 0 "#PWR0157" H 9400 11750 50  0001 C CNN
+F 1 "GND" H 9405 11827 50  0000 C CNN
+F 2 "" H 9400 12000 50  0001 C CNN
+F 3 "" H 9400 12000 50  0001 C CNN
+	1    9400 12000
 	1    0    0    -1
 $EndComp
@@
 	7550 9750 7550 9950
 Wire Wire Line
-	7550 9950 9600 9950
+	7550 9950 9250 9950
 Wire Wire Line
 	9600 10050 9600 9950
@@
 	1    0    0    -1
 $EndComp
-Text GLabel 10700 13500 0    50   Input ~ 0
-ESP_EN
 Wire Wire Line
 	10700 13500 10900 13500
 Connection ~ 10900 13500
-$Comp
-L Switch:SW_Push SW1
-U 1 1 5C3A2A38
-P 10900 14000
-F 0 "SW1" V 10854 14148 50  0000 L CNN
-F 1 "SW_Push" V 10945 14148 50  0000 L CNN
-F 2 "digikey-footprints:Switch_Tactile_SMD_B3U-1000P" H 10900 14200 50  0001 C CNN
-F 3 "" H 10900 14200 50  0001 C CNN
-	1    10900 14000
-	0    1    1    0
-$EndComp
 $Comp
 L power:GND #PWR0129
@@
 Text GLabel 15550 14500 2    50   Input ~ 0
 ESP_GPIO_0
+Wire Wire Line
+	9400 11100 9250 11100
+Wire Wire Line
+	9250 11100 9250 9950
+Connection ~ 9250 9950
+Wire Wire Line
+	9250 9950 9600 9950
+$Comp
+L Device:LED D14
+U 1 1 5C13D733
+P 12450 14000
+F 0 "D14" V 12488 13883 50  0000 R CNN
+F 1 "LED" V 12397 13883 50  0000 R CNN
+F 2 "LEDs:LED_1206" H 12450 14000 50  0001 C CNN
+F 3 "~" H 12450 14000 50  0001 C CNN
+	1    12450 14000
+	0    1    -1   0
+$EndComp
+$Comp
+L Device:Q_NMOS_GSD Q11
+U 1 1 5C13D739
+P 12550 14650
+F 0 "Q11" H 12755 14696 50  0000 L CNN
+F 1 "Q_NMOS_GSD" H 12755 14605 50  0000 L CNN
+F 2 "TO_SOT_Packages_SMD:SOT-323_SC-70" H 12750 14750 50  0001 C CNN
+F 3 "~" H 12550 14650 50  0001 C CNN
+	1    12550 14650
+	-1   0    0    -1
+$EndComp
+$Comp
+L Device:R R29
+U 1 1 5C13D73F
+P 12450 14300
+F 0 "R29" H 12520 14346 50  0000 L CNN
+F 1 "330R" H 12520 14255 50  0000 L CNN
+F 2 "Resistors_SMD:R_0603" V 12380 14300 50  0001 C CNN
+F 3 "~" H 12450 14300 50  0001 C CNN
+	1    12450 14300
+	-1   0    0    -1
+$EndComp
+$Comp
+L Device:R R30
+U 1 1 5C13D745
+P 12750 14800
+F 0 "R30" H 12820 14846 50  0000 L CNN
+F 1 "10K" H 12820 14755 50  0000 L CNN
+F 2 "Resistors_SMD:R_0603" V 12680 14800 50  0001 C CNN
+F 3 "~" H 12750 14800 50  0001 C CNN
+	1    12750 14800
+	-1   0    0    -1
+$EndComp
+Wire Wire Line
+	12750 14950 12450 14950
+Wire Wire Line
+	12450 14950 12450 14850
+Wire Wire Line
+	13700 14650 12750 14650
+Connection ~ 12750 14650
+$Comp
+L power:+3.3V #PWR0130
+U 1 1 5C13D750
+P 12450 13850
+F 0 "#PWR0130" H 12450 13700 50  0001 C CNN
+F 1 "+3.3V" V 12465 13978 50  0000 L CNN
+F 2 "" H 12450 13850 50  0001 C CNN
+F 3 "" H 12450 13850 50  0001 C CNN
+	1    12450 13850
+	-1   0    0    -1
+$EndComp
+$Comp
+L power:GND #PWR0131
+U 1 1 5C13D756
+P 12450 14950
+F 0 "#PWR0131" H 12450 14700 50  0001 C CNN
+F 1 "GND" H 12455 14777 50  0000 C CNN
+F 2 "" H 12450 14950 50  0001 C CNN
+F 3 "" H 12450 14950 50  0001 C CNN
+	1    12450 14950
+	-1   0    0    -1
+$EndComp
+Connection ~ 12450 14950
+NoConn ~ 15550 13800
+Text GLabel 10700 13500 0    50   Input ~ 0
+ESP_EN
+$Comp
+L power:+3.3V #PWR0132
+U 1 1 5C1DABDA
+P 18200 5150
+F 0 "#PWR0132" H 18200 5000 50  0001 C CNN
+F 1 "+3.3V" H 18215 5323 50  0000 C CNN
+F 2 "" H 18200 5150 50  0001 C CNN
+F 3 "" H 18200 5150 50  0001 C CNN
+	1    18200 5150
+	1    0    0    -1
+$EndComp
+$Comp
+L Device:R R31
+U 1 1 5C1DABE0
+P 18200 5300
+F 0 "R31" H 18270 5346 50  0000 L CNN
+F 1 "12k" H 18270 5255 50  0000 L CNN
+F 2 "Resistors_SMD:R_0603" V 18130 5300 50  0001 C CNN
+F 3 "~" H 18200 5300 50  0001 C CNN
+	1    18200 5300
+	1    0    0    -1
+$EndComp
+$Comp
+L Device:R R32
+U 1 1 5C1DABE6
+P 18200 5600
+F 0 "R32" H 18270 5646 50  0000 L CNN
+F 1 "470R" H 18270 5555 50  0000 L CNN
+F 2 "Resistors_SMD:R_0603" V 18130 5600 50  0001 C CNN
+F 3 "~" H 18200 5600 50  0001 C CNN
+	1    18200 5600
+	1    0    0    -1
+$EndComp
+Wire Wire Line
+	16250 5450 18200 5450
+Connection ~ 18200 5450
+$Comp
+L power:GND #PWR0133
+U 1 1 5C1DABF4
+P 18200 6150
+F 0 "#PWR0133" H 18200 5900 50  0001 C CNN
+F 1 "GND" H 18205 5977 50  0000 C CNN
+F 2 "" H 18200 6150 50  0001 C CNN
+F 3 "" H 18200 6150 50  0001 C CNN
+	1    18200 6150
+	1    0    0    -1
+$EndComp
+$Comp
+L switches_mdg:SW_Push SW2
+U 1 1 5C2268DF
+P 18200 5950
+F 0 "SW2" V 18154 6098 50  0000 L CNN
+F 1 "SW_Push" V 18245 6098 50  0000 L CNN
+F 2 "switches_mdg:Switch_Tactile_6x6mm_Vertical_SMD_MJTP1230" H 18200 6150 50  0001 C CNN
+F 3 "" H 18200 6150 50  0001 C CNN
+	1    18200 5950
+	0    1    1    0
+$EndComp
+$Comp
+L switches_mdg:SW_Push SW1
+U 1 1 5C22BD10
+P 10900 14000
+F 0 "SW1" V 10854 14148 50  0000 L CNN
+F 1 "SW_Push" V 10945 14148 50  0000 L CNN
+F 2 "switches_mdg:Switch_Tactile_6x6mm_Vertical_SMD_MJTP1230" H 10900 14200 50  0001 C CNN
+F 3 "" H 10900 14200 50  0001 C CNN
+	1    10900 14000
+	0    1    1    0
+$EndComp
 $EndSCHEMATC

Commit message: worked on layout, created board outline, started working on fitting the input, esp32, and stm32 sections together
Parts:
- removed J5: Conn_02x04_Top_Bottom, Pin_Headers:Pin_Header_Straight_2x04_Pitch2.54mm, symbol Connector_Generic:Conn_02x04_Top_Bottom
- added J5: Conn_02x04_Odd_Even, Pin_Headers:Pin_Header_Straight_2x04_Pitch2.54mm, symbol Connector_Generic:Conn_02x04_Odd_Even
- added J6, J8: Conn_01x10, Pin_Headers:Pin_Header_Straight_1x10_Pitch2.54mm, symbol Connector_Generic:Conn_01x10
- added J7: Conn_02x05_Top_Bottom, Pin_Headers:Pin_Header_Straight_2x05_Pitch2.54mm, symbol Connector_Generic:Conn_02x05_Top_Bottom
- SW1: Part Number (none) -> 1825910-6
Connections:
- wire segments 210 -> 309
Other:
- moved on the sheet: D14, Q11, R29, R30

Commit message: reworked layout of esp32 section
Parts:
- removed J3: Conn_02x08_Top_Bottom, Pin_Headers:Pin_Header_Straight_2x08_Pitch2.54mm, symbol Connector_Generic:Conn_02x08_Top_Bottom
- removed J6, J8: Conn_01x10, Pin_Headers:Pin_Header_Straight_1x10_Pitch2.54mm, symbol Connector_Generic:Conn_01x10
- removed J7: Conn_02x05_Top_Bottom, Pin_Headers:Pin_Header_Straight_2x05_Pitch2.54mm, symbol Connector_Generic:Conn_02x05_Top_Bottom
- added J3: Conn_02x08_Odd_Even, Pin_Headers:Pin_Header_Straight_2x08_Pitch2.54mm, symbol Connector_Generic:Conn_02x08_Odd_Even
- added J6, J7: Conn_01x15, Pin_Headers:Pin_Header_Straight_1x15_Pitch2.54mm, symbol Connector_Generic:Conn_01x15
- Q10, Q9: footprint TO_SOT_Packages_SMD:SOT-323_SC-70 -> TO_SOT_Packages_SMD:SOT-23
Connections:
- net labels added: CLK, CMD, IO12, IO13, IO14, IO15, IO16, IO17, IO18, IO19, IO2, IO21, IO22, IO23, IO25, IO26, IO27, IO32, IO33, IO35, IO4, IO5, SD0, SD1, SD2, SD3, SENSOR_VN, SENSOR_VP
- wire segments 309 -> 244
Other:
- moved on the sheet: J5, R27, R28, SW1

Commit message: layout almost done, changing my mind, getting rid of esp32, usb section
Parts:
- removed Q10, Q9: 2N2219, TO_SOT_Packages_SMD:SOT-23, symbol Transistor_BJT:2N2219
- added C19, C20: 0.1uF, Capacitors_SMD:C_0603, symbol Device:C
- added J10, J11, J8, J9: Conn_01x15, Pin_Headers:Pin_Header_Straight_1x15_Pitch2.54mm, symbol Connector_Generic:Conn_01x15
- added Q10, Q9: Q_NPN_BEC, TO_SOT_Packages_SMD:SOT-23, symbol Device:Q_NPN_BEC
- R25, R26: value 12k -> 10k
Connections:
- net labels added: PA1, PA15, PA2, PA8, PB0, PB1, PB10, PB11, PB12, PB13, PB14, PB15, PB2, PB4, PB5, PB6, PB7, PB8, PB9, PC0, PC1, PC10, PC11, PC12, PC13, PC14, PC15, PC2, PC4, PC5, PC6, PC7, PC8, PC9, PD0, PD1, PD10, PD11, PD12, PD13, PD14, PD15, PD2, PD3, PD4, PD7, PD8, PD9, PE0, PE1, PE2, PE3, PE4, PE5, PE6, PE7
- wire segments 244 -> 310
Other:
- moved on the sheet: C1, C10, C11, C12, C13, C14, C15, C16, C17, C18, C2, C3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

Commit message: Ordered PCB 12/18
Parts:
- removed C12, C13, C14, C15: C, Capacitors_SMD:C_0603, symbol Device:C
- removed C19: 0.1uF, Capacitors_SMD:C_0603, symbol Device:C
- removed D1: SP0502BAHT, TO_SOT_Packages_SMD:SOT-23, symbol Power_Protection:SP0502BAHT
- removed D14, D2, D3: LED, LEDs:LED_1206, symbol Device:LED
- removed J1: USB_B_Mini, Connectors:USB_Mini-B, symbol Connector:USB_B_Mini
- removed J10, J11, J6, J7, J8, J9: Conn_01x15, Pin_Headers:Pin_Header_Straight_1x15_Pitch2.54mm, symbol Connector_Generic:Conn_01x15
- removed J3: Conn_02x08_Odd_Even, Pin_Headers:Pin_Header_Straight_2x08_Pitch2.54mm, symbol Connector_Generic:Conn_02x08_Odd_Even
- removed J4: Conn_01x10, Pin_Headers:Pin_Header_Straight_1x10_Pitch2.54mm, symbol Connector_Generic:Conn_01x10
- removed J5: Conn_02x04_Odd_Even, Pin_Headers:Pin_Header_Straight_2x04_Pitch2.54mm, symbol Connector_Generic:Conn_02x04_Odd_Even
- removed Q10, Q9: Q_NPN_BEC, TO_SOT_Packages_SMD:SOT-23, symbol Device:Q_NPN_BEC
- removed Q11: Q_NMOS_GSD, TO_SOT_Packages_SMD:SOT-323_SC-70, symbol Device:Q_NMOS_GSD
- removed R25, R26: 10k, Resistors_SMD:R_0603, symbol Device:R
- removed R27: 12k, Resistors_SMD:R_0603, symbol Device:R
- removed R28: 470R, Resistors_SMD:R_0603, symbol Device:R
- removed R29, R5, R6: 330R, Resistors_SMD:R_0603, symbol Device:R
- removed R30: 10K, Resistors_SMD:R_0603, symbol Device:R
- removed R7, R8: 0R, Resistors_SMD:R_0603, symbol Device:R
- removed SW1: SW_Push, switches_mdg:Switch_Tactile_6x6mm_Vertical_SMD_MJTP1230, symbol switches_mdg:SW_Push
- removed U1: FT232RL, Housings_SSOP:TSSOP-28_4.4x9.7mm_Pitch0.65mm, symbol Interface_USB:FT232RL
- removed U5: ESP32-WROOM, ESP32-footprints-Lib:ESP32-WROOM, symbol ESP32-footprints-Shem-Lib:ESP32-WROOM
- added J1: Conn_01x04, Pin_Headers:Pin_Header_Straight_1x04_Pitch2.54mm, symbol Connector_Generic:Conn_01x04
- added J10: Conn_01x03, Pin_Headers:Pin_Header_Straight_1x03_Pitch2.54mm, symbol Connector_Generic:Conn_01x03
- added J11: Conn_01x05, Pin_Headers:Pin_Header_Straight_1x05_Pitch2.54mm, symbol Connector_Generic:Conn_01x05
- added J12: Conn_01x07, Pin_Headers:Pin_Header_Straight_1x07_Pitch2.54mm, symbol Connector_Generic:Conn_01x07
- added J13, J4, J5, J6, J7: Conn_01x06, Pin_Headers:Pin_Header_Straight_1x06_Pitch2.54mm, symbol Connector_Generic:Conn_01x06
- added J14: Conn_01x30, Pin_Headers:Pin_Header_Straight_1x30_Pitch2.54mm, symbol Connector_Generic:Conn_01x30
- added J3, J9: Conn_01x08, Pin_Headers:Pin_Header_Straight_1x08_Pitch2.54mm, symbol Connector_Generic:Conn_01x08
- C1, C10, C11, C41, C5, C6, C7, C8, C9: value C -> .1uF
- C2, C3: value C -> 9pF
- C4: value C -> 1uF
- R3, R4: value 0R -> 10K
- R31: value 12k -> 10k
Connections:
- net PA8 is gone; now on net STATUS_BIT7: U3.67 (PA8)
- net PB6 is gone; now on net I2C1_SCL: U3.92 (PB6)
- net PB7 is gone; now on net I2C1_SDA: U3.93 (PB7)
- net PC6 is gone; now on net STATUS_BIT3: U3.63 (PC6)
- net PC7 is gone; now on net STATUS_BIT4: U3.64 (PC7)
- net PC8 is gone; now on net STATUS_BIT5: U3.65 (PC8)
- net PC9 is gone; now on net STATUS_BIT6: U3.66 (PC9)
- net PD13 is gone; now on net STATUS_BIT0: U3.60 (PD13)
- net PD14 is gone; now on net STATUS_BIT1: U3.61 (PD14)
- net PD15 is gone; now on net STATUS_BIT2: U3.62 (PD15)
- net +3V3: now also R3.1, R4.1, J12.6 (Pin_6), J13.5 (Pin_5), J4.5 (Pin_5), J5.5 (Pin_5), J6.5 (Pin_5), J7.5 (Pin_5)
- net +5V: now also J3.1 (Pin_1), J4.4 (Pin_4), J5.4 (Pin_4), J6.4 (Pin_4), J7.4 (Pin_4)
- net FTDI_CTS: now also J3.7 (Pin_7); no longer R4.1
- net FTDI_DCD: now also J3.4 (Pin_4)
- net FTDI_DCR: now also J3.3 (Pin_3)
- net FTDI_RI: now also J3.2 (Pin_2)
- net FTDI_ST_DTR: now also J3.5 (Pin_5)
- net FTDI_ST_RTS: now also J3.6 (Pin_6)
- net FTDI_ST_RXD: now also J1.4 (Pin_4)
- net FTDI_ST_TXD: now also J1.3 (Pin_3)
- net GND: now also J1.1 (Pin_1), J12.7 (Pin_7), J13.6 (Pin_6), J3.8 (Pin_8), J4.6 (Pin_6), J5.6 (Pin_6), J6.6 (Pin_6), J7.6 (Pin_6)
- net PA1: now also J14.27 (Pin_27)
- net PA2: now also J14.26 (Pin_26)
- net PB0: now also J14.23 (Pin_23)
- net PB1: now also J14.22 (Pin_22)
- net PB10: now also J14.11 (Pin_11)
- net PB11: now also J14.10 (Pin_10)
- net PB12: now also J14.9 (Pin_9)
- net PB13: now also J14.8 (Pin_8)
- net PB14: now also J14.7 (Pin_7)
- net PB15: now also J14.6 (Pin_6)
- net PB2: now also J14.21 (Pin_21)
- net PB4: now also J11.1 (Pin_1)
- net PB8: now also J11.2 (Pin_2)
- net PB9: now also J11.3 (Pin_3)
- net PC0: now also J14.30 (Pin_30)
- net PC1: now also J14.29 (Pin_29)
- net PC13: now also J9.3 (Pin_3)
- net PC14: now also J9.2 (Pin_2)
- net PC15: now also J9.1 (Pin_1)
- net PC2: now also J14.28 (Pin_28)
- net PC4: now also J14.25 (Pin_25)
- net PC5: now also J14.24 (Pin_24)
- net PD0: now also J10.1 (Pin_1)
- net PD1: now also J10.2 (Pin_2)
- net PD10: now also J14.3 (Pin_3)
- net PD11: now also J14.2 (Pin_2)
- net PD12: now also J14.1 (Pin_1)
- net PD2: now also J10.3 (Pin_3)
- net PD8: now also J14.5 (Pin_5)
- net PD9: now also J14.4 (Pin_4)
- net PE0: now also J11.4 (Pin_4)
- net PE1: now also J11.5 (Pin_5)
- net PE2: now also J9.8 (Pin_8)
- net PE3: now also J9.7 (Pin_7)
- net PE4: now also J9.6 (Pin_6)
- net PE5: now also J9.5 (Pin_5)
- net PE6: now also J9.4 (Pin_4)
- net PE7: now also J14.20 (Pin_20)
- net STATUS_BIT0: no longer U3.39 (PE8)
- net STATUS_BIT1: no longer U3.40 (PE9)
- net STATUS_BIT2: no longer U3.41 (PE10)
- net STATUS_BIT3: no longer U3.42 (PE11)
- net STATUS_BIT4: no longer U3.43 (PE12)
- net STATUS_BIT5: no longer U3.44 (PE13)
- net STATUS_BIT6: no longer U3.45 (PE14)
- net STATUS_BIT7: no longer U3.46 (PE15)
- net I2C1_SDA: now reaches R4.2
- net I2C1_SDA: now also J4.1 (Pin_1), J5.1 (Pin_1), J6.1 (Pin_1), J7.1 (Pin_1)
- net I2C1_SCL: now reaches R3.2
- net I2C1_SCL: now also J4.2 (Pin_2), J5.2 (Pin_2), J6.2 (Pin_2), J7.2 (Pin_2)
- net PA15 renamed SPI3_NSS
- net SPI3_NSS: now also J13.1 (Pin_1)
- net PB5 renamed I2C1_SMBA
- net I2C1_SMBA: now also J4.3 (Pin_3), J5.3 (Pin_3), J6.3 (Pin_3), J7.3 (Pin_3)
- net PC10 renamed SPI3_SCK
- net SPI3_SCK: now also J13.2 (Pin_2)
- net PC11 renamed SPI3_MISO
- net SPI3_MISO: now also J13.3 (Pin_3)
- net PC12 renamed SPI3_MOSI
- net SPI3_MOSI: now also J13.4 (Pin_4)
- net PD3 renamed USART2_CTS
- net USART2_CTS: now also J12.5 (Pin_5)
- net PD4 renamed USART2_RTS
- net USART2_RTS: now also J12.4 (Pin_4)
- net PD7 renamed USART2_CK
- net USART2_CK: now also J12.1 (Pin_1)
- net ST_ESP_RXD renamed USART2_TX
- net USART2_TX: now also J12.3 (Pin_3)
- net ST_ESP_TXD renamed USART2_RX
- net USART2_RX: now also J12.2 (Pin_2)
- net ST_MISO renamed SPI1_MISO
- net ST_MOSI renamed SPI1_MOSI
- net ST_SCK renamed SPI1_SCK
- new net PE10: J14.17 (Pin_17), U3.41 (PE10)
- new net PE11: J14.16 (Pin_16), U3.42 (PE11)
- new net PE12: J14.15 (Pin_15), U3.43 (PE12)
- new net PE13: J14.14 (Pin_14), U3.44 (PE13)
- new net PE14: J14.13 (Pin_13), U3.45 (PE14)
- new net PE15: J14.12 (Pin_12), U3.46 (PE15)
- new net PE8: J14.19 (Pin_19), U3.39 (PE8)
- new net PE9: J14.18 (Pin_18), U3.40 (PE9)
Other:
- moved on the sheet: C1, C10, C11, C16, C17, C18, C2, C20, C3, C38, C39, C4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

Commit message: began simplifying, switching to STM32F405 series
Parts:
- removed C1: .1uF, Capacitors_SMD:C_0603, symbol Device:C
- removed C17: 0.1uF, Capacitors_SMD:C_0603, symbol Device:C
- removed C18: 10uF, Capacitors_SMD:C_0603, symbol Device:C
- removed J10: Conn_01x03, Pin_Headers:Pin_Header_Straight_1x03_Pitch2.54mm, symbol Connector_Generic:Conn_01x03
- removed J11: Conn_01x05, Pin_Headers:Pin_Header_Straight_1x05_Pitch2.54mm, symbol Connector_Generic:Conn_01x05
- removed J14: Conn_01x30, Pin_Headers:Pin_Header_Straight_1x30_Pitch2.54mm, symbol Connector_Generic:Conn_01x30
- removed J9: Conn_01x08, Pin_Headers:Pin_Header_Straight_1x08_Pitch2.54mm, symbol Connector_Generic:Conn_01x08
- removed R10, R34, R35, R36, R49, R9: 0R, Resistors_SMD:R_0603, symbol Device:R
- removed U2: W25Q128JV-DTR, Housings_SOIC:SOIC-8_3.9x4.9mm_Pitch1.27mm, symbol flash_memory_mdg:W25Q128JV-DTR
- removed U4: LD1117S33TR, TO_SOT_Packages_SMD:SOT-223, symbol Voltage_Regulators:LD1117S33TR
- added C?: 0.1uF, Capacitors_SMD:C_0603, symbol Device:C
- added C? (x6): .1uF, Capacitors_SMD:C_0603, symbol Device:C
- added C? (x2): 9pF, Capacitors_SMD:C_0603, symbol Device:C
- added J? (x2): Conn_01x03, symbol Connector_Generic:Conn_01x03
- added R? (x3): 10k, Resistors_SMD:R_0603, symbol Device:R
- added R? (x2): 510, Resistors_SMD:R_0603, symbol Device:R
- added R?: 1MR, Resistors_SMD:R_0603, symbol Device:R
- added SW?: SW_Push, switches_mdg:Switch_Tactile_6x6mm_Vertical_SMD_MJTP1230, symbol switches_mdg:SW_Push
- added U?: STM32F405RGTx, Package_QFP:LQFP-64_10x10mm_P0.5mm, symbol MCU_ST_STM32F4:STM32F405RGTx
- added Y?: Crystal_GND24, Crystals:Crystal_SMD_SeikoEpson_TSX3225-4pin_3.2x2.5mm, symbol Device:Crystal_GND24
Connections:
- net +3V3: now also C?.2, C?.2, C?.2, C?.2, C?.2, C?.2, R?.1, R?.1, R?.1, U?.1 (VBAT), U?.13 (VDDA), U?.19 (VDD), U?.32 (VDD), U?.48 (VDD), U?.64 (VDD)
- net FTDI_CTS: now also U?.45 (PA12)
- net FTDI_ST_RTS: now also U?.44 (PA11)
- net FTDI_ST_RXD: now also U?.42 (PA9)
- net FTDI_ST_TXD: now also U?.43 (PA10)
- net GND: now also C?.1, C?.1, C?.1, C?.1, C?.1, C?.1, C?.1, C?.2, C?.2, R?.1, R?.1, SW?.3 (2), U?.12 (VSSA), U?.18 (VSS), U?.63 (VSS), Y?.1, Y?.3
- net I2C1_SCL: now also U?.58 (PB6)
- net I2C1_SDA: now also U?.59 (PB7)
- net I2C1_SMBA: now also U?.57 (PB5)
- net SPI1_MISO: now also U?.22 (PA6)
- net SPI1_MOSI: now also U?.23 (PA7)
- net SPI1_SCK: now also U?.21 (PA5)
- net at R31.2, R32.1: now also U?.14 (PA0); no longer U3.23 (PA0)
- new net: J?.2 (Pin_2), U?.28 (PB2)
- new net: C?.1, R?.1, U?.5 (PH0), Y?.2
- new net: C?.1, R?.2, U?.6 (PH1), Y?.4
- new net: J?.2 (Pin_2), U?.60 (BOOT0)
- new net: C?.2, R?.2, SW?.1, U?.7 (NRST)
- new net: J?.3 (Pin_3), R?.2 (x2)
- new net: J?.1 (Pin_1), R?.2 (x2)
- new net SPI1_NSS: U?.20 (PA4)
Other:
- moved on the sheet: C20, R31, R32, SW2
