File: stm32 prototype.sch (KiCad schematic (older format))
At the start: 102 parts, among them J1 Conn_01x04, J12 Conn_01x07, J13 Conn_01x06, J2 Conn_01x06, J3 Conn_01x08, J4 Conn_01x06, J5 Conn_01x06, J6 Conn_01x06, J7 Conn_01x06, Q1 Q_NMOS_GSD, Q2 Q_NMOS_GSD, Q3 Q_NMOS_GSD, Q4 Q_NMOS_GSD, Q5 Q_NMOS_GSD, Q6 Q_NMOS_GSD, Q7 Q_NMOS_GSD, Q8 Q_NMOS_GSD, SW2 SW_Push, U3 STM32F407VGTx, U7 TPS62203DBVR, Y1 Crystal_GND24

Commit message: pushed change to stm32f405 to pcb
Parts:
- removed J2: Conn_01x06, Pin_Headers:Pin_Header_Straight_1x06_Pitch2.54mm, symbol Connector_Generic:Conn_01x06
- removed R40, R41, R42, R43, R44, R45: 0R, Resistors_SMD:R_0603, symbol Device:R
- removed R? (x2): 510, Resistors_SMD:R_0603, symbol Device:R
- added C1: 4.7uF, Capacitors_SMD:C_0603, symbol Device:C
- added C13, C14: 2.2uF, Capacitors_SMD:C_0603, symbol Device:C
- added J2: Conn_02x05_Odd_Even, Pin_Headers:Pin_Header_Straight_2x05_Pitch1.27mm_SMD, symbol Connector_Generic:Conn_02x05_Odd_Even
- added J8: Conn_ARM_JTAG_SWD_10, Pin_Headers:Pin_Header_Straight_2x05_Pitch1.27mm_SMD, symbol Connector:Conn_ARM_JTAG_SWD_10
- gave numbers to parts that had none: 18
Connections:
- net +3V3: now also J10.3 (Pin_3), J9.3 (Pin_3), C1.2, J2.1 (Pin_1), J8.1 (VCC); no longer R6.1, R8.1
- net GND: now also J10.1 (Pin_1), J9.1 (Pin_1), C1.1, C13.1, C14.1, J2.3 (Pin_3), J2.5 (Pin_5), J2.9 (Pin_9), J8.3 (GND), J8.5 (GND), J8.9 (GNDDetect)
- net NRST: now also J2.10 (Pin_10), J8.10 (~RESET~)
- net SWO: now also J2.6 (Pin_6), J8.6 (SWO/TDO)
- net TCK_SWCLK: now also J2.4 (Pin_4), J8.4 (SWDCLK/TCK)
- net TMS_SWDIO: now also J2.2 (Pin_2), J8.2 (SWDIO/TMS)
- net at U1.28 (PB2): now also R8.1; no longer J10.2 (Pin_2)
- net at U1.31 (VCAP_1): now also C13.2
- net at U1.47 (VCAP_2): now also C14.2
- net at U1.60 (BOOT0): now also R6.1; no longer J9.2 (Pin_2)
- net at R6.2: now also J9.2 (Pin_2); no longer J9.3 (Pin_3)
- net at R8.2: now also J10.2 (Pin_2); no longer J10.3 (Pin_3)
Other:
- note removed: "SWD PROGRAMMING\nHEADER"
- moved on the sheet: J1, J3, R6, R8
